File: KiCad/Binary-G2-Revised.kicad_pcb (KiCad board)
At the start: 2 copper layers, 75 x 50 mm, 90 parts, among them J1 USB_C_Receptacle_PowerOnly_6P, J2 Conn_01x01, J3 Conn_01x01, SW1 PTH_RA_7.4x4.3mm, SW2 PTH_RA_7.4x4.3mm, SW3 PTH_RA_7.4x4.3mm, SW4 SW_SPDT, U1 74HC4060, U10 BQ21040DBV, U12 MCP65R41-2402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

Commit message: Update with minimum layout
Needs a lot more work.
Routing:
- net VDD: track 74.9 -> 237.3 mm, vias 0 -> 18
- net /SIN: track 0.00 -> 62.1 mm, vias 0 -> 6
- net Net-(D5-A): track 0.00 -> 49.5 mm, vias 0 -> 2
- net Net-(D2-A): track 4.07 -> 45.1 mm, vias 0 -> 2
- net Net-(D11-A): track 0.00 -> 37.4 mm, vias 0 -> 4
- net Net-(U8B-MR): track 0.00 -> 37.1 mm, vias 0 -> 3
- net /Hin: track 0.00 -> 33.5 mm
- net Net-(U9B-MR): track 0.08 -> 33.1 mm
- net Net-(D6-A): track 0.00 -> 30.9 mm, vias 0 -> 3
- net Net-(D7-A): track 0.00 -> 30.6 mm, vias 0 -> 2
- net Net-(U7B-MR): track 0.00 -> 29.1 mm
- net Net-(U9A-MR): track 4.95 -> 33.9 mm, vias 0 -> 2
- net Net-(D3-K): track 10.2 -> 38.5 mm, vias 0 -> 1
- net Net-(D12-A): track 0.00 -> 25.1 mm, vias 0 -> 3
- net Net-(D14-A): track 0.00 -> 24.6 mm, vias 0 -> 1
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
Commit message: Quick Update Documentation
Parts:
- moved D11 91.6 mm to (68.6, 53.0)
- moved D14 91.6 mm to (98.1, 53.0)
- moved D3 91.6 mm to (98.1, 32.7)
- moved D5 91.6 mm to (68.6, 42.8)
- moved D8 91.6 mm to (98.1, 42.8)
- moved R16 91.6 mm to (97.0, 68.3)
- moved R19 91.6 mm to (50.8, 24.5)
- moved R34 91.6 mm to (46.8, 65.1)
- moved R8 91.6 mm to (99.0, 68.3)
- moved U7 91.6 mm to (98.1, 60.6)
- moved C1 91.6 mm to (93.4, 24.3)
- moved C11 91.6 mm to (40.5, 49.3)
- moved C3 91.6 mm to (59.1, 24.3)
- moved C4 91.6 mm to (44.5, 28.9)
- moved C5 91.6 mm to (40.0, 32.7)
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Routing:
- net GND: track 15.6 -> 27.5 mm, vias 8 -> 12
