File: KiCad/Binary-G2-Revised.kicad_sch (KiCad schematic)
At the start: 91 parts, among them J1 USB_C_Receptacle_PowerOnly_6P, J2 Conn_01x01, J3 Conn_01x01, SW1 PTH_RA_7.4x4.3mm, SW2 PTH_RA_7.4x4.3mm, SW3 PTH_RA_7.4x4.3mm, SW4 SW_SPDT, U1 74HC4060, U10 BQ21040DBV, U12 MCP65R41-2402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

Commit message: Update with minimum layout
Needs a lot more work.
Other:
- company: (none) -> Foxhood Designs
- title: (none) -> BCD Clock
Changed lines of the file:
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@@
 	(generator_version "9.0")
 	(paper "A3")
+	(title_block
+		(title "BCD Clock")
+		(date "2025-02-24")
+		(rev "2")
+		(company "Foxhood Designs")
+		(comment 1 "TODO: Double Check logic")
+		(comment 2 "TODO: Optimize PCB Layout for consistency.")
+	)
 	(junction
 		(at 73.66 248.92)

Commit message: Quick Update Documentation
Other:
- moved on the sheet: BT1, C11, D1, D10, D11, D12, D13, D14, D15, D16, D17, D18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
